Commit message: Replace RTK2026 workspace with RTK2026-2

File: src/rtk2026_description/urdf/rtk2026.urdf.xacro (robot description, xacro)
@@ -1,5 +1,106 @@
 <?xml version="1.0"?>
 <robot xmlns:xacro="http://www.ros.org/wiki/xacro" name="rtk2026">
-  <xacro:include filename="rtk2026_macro.xacro"/>
-  <xacro:rtk2026_macro prefix="" />
+  <!-- ━━━━━━━━━━━━━━━━━━━━━━━━━━━━━━━━━━━━━━━━━━━━━━━━
+       Параметры робота
+       Корпус: 300×250×113 мм, дифференциальный привод
+       Колёса: диаметр 51.7 мм, расстояние между колёсами 212.3 мм
+       ━━━━━━━━━━━━━━━━━━━━━━━━━━━━━━━━━━━━━━━━━━━━━━━━ -->
+  <xacro:property name="base_length"     value="0.300"/>
+  <xacro:property name="base_width"      value="0.240"/>
+  <xacro:property name="base_height"     value="0.113"/>
+  <xacro:property name="wheel_radius"    value="0.02585"/>  <!-- 51.7 мм / 2 -->
+  <xacro:property name="wheel_width"     value="0.030"/>
+  <xacro:property name="wheel_sep"       value="0.2123"/>   <!-- между центрами колёс -->
+  <xacro:property name="base_z_offset"   value="0.0565"/>   <!-- центр корпуса над полом -->
+  <!-- ── base_footprint — точка на полу под роботом ── -->
+  <link name="base_footprint"/>
+  <joint name="base_footprint_joint" type="fixed">
+    <parent link="base_footprint"/>
+    <child link="base_link"/>
+    <origin xyz="0 0 ${base_z_offset}" rpy="0 0 0"/>
+  </joint>
+  <!-- ── base_link — центр корпуса ── -->
+  <link name="base_link">
+    <visual>
+      <geometry>
+        <box size="${base_length} ${base_width} ${base_height}"/>
+      </geometry>
+      <material name="base_grey">
+        <color rgba="0.4 0.4 0.4 1"/>
+      </material>
+    </visual>
+    <collision>
+      <geometry>
+        <box size="${base_length} ${base_width} ${base_height}"/>
+      </geometry>
+    </collision>
+    <inertial>
+      <mass value="5.0"/>
+      <inertia ixx="0.05" ixy="0" ixz="0" iyy="0.05" iyz="0" izz="0.05"/>
+    </inertial>
+  </link>
+  <!-- ── левое колесо ── -->
+  <joint name="left_wheel_joint" type="continuous">
+    <parent link="base_link"/>
+    <child link="left_wheel_link"/>
+    <origin xyz="0 ${wheel_sep/2} ${-base_z_offset + wheel_radius}" rpy="-1.5708 0 0"/>
+    <axis xyz="0 0 1"/>
+  </joint>
+  <link name="left_wheel_link">
+    <visual>
+      <geometry>
+        <cylinder radius="${wheel_radius}" length="${wheel_width}"/>
+      </geometry>
+      <material name="wheel_black">
+        <color rgba="0.1 0.1 0.1 1"/>
+      </material>
+    </visual>
+    <collision>
+      <geometry>
+        <cylinder radius="${wheel_radius}" length="${wheel_width}"/>
+      </geometry>
+    </collision>
+    <inertial>
+      <mass value="0.3"/>
+      <inertia ixx="0.001" ixy="0" ixz="0" iyy="0.001" iyz="0" izz="0.001"/>
+    </inertial>
+  </link>
+  <!-- ── правое колесо ── -->
+  <joint name="right_wheel_joint" type="continuous">
+    <parent link="base_link"/>
+    <child link="right_wheel_link"/>
+    <origin xyz="0 ${-wheel_sep/2} ${-base_z_offset + wheel_radius}" rpy="-1.5708 0 0"/>
+    <axis xyz="0 0 1"/>
+  </joint>
+  <link name="right_wheel_link">
+    <visual>
+      <geometry>
+        <cylinder radius="${wheel_radius}" length="${wheel_width}"/>
+      </geometry>
+      <material name="wheel_black"/>
+    </visual>
+    <collision>
+      <geometry>
+        <cylinder radius="${wheel_radius}" length="${wheel_width}"/>
+      </geometry>
+    </collision>
+    <inertial>
+      <mass value="0.3"/>
+      <inertia ixx="0.001" ixy="0" ixz="0" iyy="0.001" iyz="0" izz="0.001"/>
+    </inertial>
+  </link>
+  <!-- ── лидар — спереди сверху корпуса ── -->
+  <joint name="lidar_joint" type="fixed">
+    <parent link="base_link"/>
+    <child link="lidar_link"/>
+    <origin xyz="0.15 0 0.08" rpy="0 0 0"/>
+  </joint>
+  <link name="lidar_link"/>
+  <!-- ── IMU ── -->
+  <joint name="imu_joint" type="fixed">
+    <parent link="base_link"/>
+    <child link="imu_link"/>
+    <origin xyz="0 0 0.04" rpy="0 0 0"/>
+  </joint>
+  <link name="imu_link"/>
 </robot>

Commit message: Add sign detection pipeline and sign-aware routing

File: src/rtk2026_description/urdf/rtk2026.urdf.xacro (robot description, xacro)
@@ -97,4 +97,29 @@
   </joint>
   <link name="lidar_link"/>
+  <!-- ── фронтальная камера ── -->
+  <joint name="camera_joint" type="fixed">
+    <parent link="base_link"/>
+    <child link="camera_link"/>
+    <origin xyz="0.12 0 0.06" rpy="0 0 0"/>
+  </joint>
+  <link name="camera_link">
+    <visual>
+      <geometry>
+        <box size="0.035 0.035 0.035"/>
+      </geometry>
+      <material name="camera_black">
+        <color rgba="0.12 0.12 0.12 1"/>
+      </material>
+    </visual>
+    <collision>
+      <geometry>
+        <box size="0.035 0.035 0.035"/>
+      </geometry>
+    </collision>
+    <inertial>
+      <mass value="0.05"/>
+      <inertia ixx="0.0001" ixy="0" ixz="0" iyy="0.0001" iyz="0" izz="0.0001"/>
+    </inertial>
+  </link>
   <!-- ── IMU ── -->
   <joint name="imu_joint" type="fixed">

File: src/rtk2026_description/urdf/rtk2026_gazebo.urdf.xacro (robot description, xacro)
@@ -131,4 +131,25 @@
     <child link="lidar_link"/>
     <origin xyz="0.1 0 ${base_height + 0.02}" rpy="0 0 0"/>
+  </joint>
+  <!-- ── фронтальная камера ── -->
+  <link name="camera_link">
+    <inertial>
+      <mass value="0.05"/>
+      <inertia ixx="0.0001" ixy="0" ixz="0" iyy="0.0001" iyz="0" izz="0.0001"/>
+    </inertial>
+    <visual>
+      <origin xyz="0 0 0" rpy="0 0 0"/>
+      <geometry><box size="0.035 0.035 0.035"/></geometry>
+      <material name="black"/>
+    </visual>
+    <collision>
+      <origin xyz="0 0 0" rpy="0 0 0"/>
+      <geometry><box size="0.035 0.035 0.035"/></geometry>
+    </collision>
+  </link>
+  <joint name="camera_joint" type="fixed">
+    <parent link="base_link"/>
+    <child link="camera_link"/>
+    <origin xyz="0.12 0 0.06" rpy="0 0 0"/>
   </joint>
   <!-- ━━━━━━━━━━━━━━━━━━━━━━━━━━━━━━━━━━━━━━━━━━━━━━━━
@@ -183,7 +204,29 @@
     </sensor>
   </gazebo>
+  <gazebo reference="camera_link">
+    <sensor name="camera" type="camera">
+      <always_on>true</always_on>
+      <visualize>false</visualize>
+      <update_rate>10</update_rate>
+      <topic>camera/image_raw</topic>
+      <camera>
+        <horizontal_fov>1.3962634</horizontal_fov>
+        <image>
+          <width>640</width>
+          <height>480</height>
+          <format>R8G8B8</format>
+        </image>
+        <clip>
+          <near>0.05</near>
+          <far>20.0</far>
+        </clip>
+        <camera_info_topic>camera/camera_info</camera_info_topic>
+      </camera>
+    </sensor>
+  </gazebo>
   <gazebo reference="base_link"><material>Gazebo/DarkGrey</material></gazebo>
   <gazebo reference="left_wheel"><material>Gazebo/Black</material></gazebo>
   <gazebo reference="right_wheel"><material>Gazebo/Black</material></gazebo>
+  <gazebo reference="camera_link"><material>Gazebo/Black</material></gazebo>
   <gazebo reference="front_caster_link">
     <material>Gazebo/White</material>

Commit message: Integrate MeArm with current RTK2026 simulation

File: src/rtk2026_description/urdf/rtk2026.urdf.xacro (robot description, xacro)
@@ -14,4 +14,5 @@
   <xacro:property name="base_z_offset"   value="0.0565"/>   <!-- центр корпуса над полом -->
   <!-- ── base_footprint — точка на полу под роботом ── -->
+  <xacro:include filename="mearm_macro.xacro"/>
   <link name="base_footprint"/>
   <joint name="base_footprint_joint" type="fixed">
@@ -129,3 +130,4 @@
   </joint>
   <link name="imu_link"/>
+  <xacro:mearm parent="base_link" mount_xyz="-0.07 -0.07 0.138"/>
 </robot>

File: src/rtk2026_description/urdf/rtk2026_gazebo.urdf.xacro (robot description, xacro)
@@ -14,4 +14,5 @@
   <xacro:property name="caster_radius" value="0.012"/>
   <xacro:property name="caster_x"      value="0.120"/>
+  <xacro:include filename="mearm_macro.xacro"/>
   <material name="grey">  <color rgba="0.4 0.4 0.4 1"/></material>
   <material name="black"> <color rgba="0.1 0.1 0.1 1"/></material>
@@ -153,4 +154,5 @@
     <origin xyz="0.12 0 0.06" rpy="0 0 0"/>
   </joint>
+  <xacro:mearm parent="base_link" mount_xyz="-0.07 -0.07 0.138"/>
   <!-- ━━━━━━━━━━━━━━━━━━━━━━━━━━━━━━━━━━━━━━━━━━━━━━━━
        Gazebo Sim (gz): привод и joint states
@@ -170,4 +172,28 @@
       <joint_name>left_wheel_joint</joint_name>
       <joint_name>right_wheel_joint</joint_name>
+      <joint_name>joint_0</joint_name>
+      <joint_name>joint_1</joint_name>
+      <joint_name>joint_2</joint_name>
+      <joint_name>joint_3</joint_name>
+    </plugin>
+    <plugin name="gz::sim::v8::systems::JointPositionController" filename="libgz-sim8-joint-position-controller-system.so">
+      <joint_name>joint_0</joint_name>
+      <topic>/model/rtk2026/joint/joint_0/0/cmd_pos</topic>
+      <p_gain>8.0</p_gain>
+    </plugin>
+    <plugin name="gz::sim::v8::systems::JointPositionController" filename="libgz-sim8-joint-position-controller-system.so">
+      <joint_name>joint_1</joint_name>
+      <topic>/model/rtk2026/joint/joint_1/0/cmd_pos</topic>
+      <p_gain>8.0</p_gain>
+    </plugin>
+    <plugin name="gz::sim::v8::systems::JointPositionController" filename="libgz-sim8-joint-position-controller-system.so">
+      <joint_name>joint_2</joint_name>
+      <topic>/model/rtk2026/joint/joint_2/0/cmd_pos</topic>
+      <p_gain>8.0</p_gain>
+    </plugin>
+    <plugin name="gz::sim::v8::systems::JointPositionController" filename="libgz-sim8-joint-position-controller-system.so">
+      <joint_name>joint_3</joint_name>
+      <topic>/model/rtk2026/joint/joint_3/0/cmd_pos</topic>
+      <p_gain>8.0</p_gain>
     </plugin>
   </gazebo>
@@ -229,4 +255,8 @@
   <gazebo reference="right_wheel"><material>Gazebo/Black</material></gazebo>
   <gazebo reference="camera_link"><material>Gazebo/Black</material></gazebo>
+  <gazebo reference="mearm_shoulder_link"><material>Gazebo/Orange</material></gazebo>
+  <gazebo reference="mearm_upper_arm_link"><material>Gazebo/Orange</material></gazebo>
+  <gazebo reference="mearm_forearm_link"><material>Gazebo/Orange</material></gazebo>
+  <gazebo reference="mearm_gripper_link"><material>Gazebo/Red</material></gazebo>
   <gazebo reference="front_caster_link">
     <material>Gazebo/White</material>
