Commit message: Описание робота, сенсоры, миры и карты
Описание приведено к габаритам платформы 310 x 246 мм. Добавлены модели
сенсоров для Gazebo: IMU, RealSense D435i и обновлённая веб-камера.

Миры: полигон 5x5 обновлён, добавлены варианты стенда с электролизными
ваннами и модульное дерево моделей к нему - ванна, платформа, задняя стена
и метка ArUco с генератором.

Bringup: конфигурация моста Gazebo вынесена в файл, добавлен лаунч
локализации на реальном роботе и отдельная сцена RViz для камеры.
Карты полигона и записанные карты лежат в maps, на них по умолчанию
ссылается запуск. Конфигурация RTAB-Map для RGBD добавлена в rtk2026_slam.

Co-Authored-By: Claude Opus 5 <noreply@anthropic.com>

File: src/rtk2026_description/urdf/rtk2026_diff_drive_sim.urdf.xacro (robot description, xacro)
@@ -21,9 +21,15 @@
     filename="$(find rtk2026_description)/urdf/sensors/imu.xacro"/>
   <xacro:include
+    filename="$(find rtk2026_description)/urdf/sensors/imu_gazebo.xacro"/>
+  <xacro:include
     filename="$(find rtk2026_description)/urdf/sensors/lidar.xacro"/>
   <xacro:include
     filename="$(find rtk2026_description)/urdf/sensors/lidar_gazebo.xacro"/>
+  <!-- Официальная геометрия и nominal extrinsics Intel RealSense D435i. -->
   <xacro:include
-    filename="$(find rtk2026_description)/urdf/sensors/webcam.xacro"/>
+    filename="$(find realsense2_description)/urdf/_d435i.urdf.xacro"/>
+  <!-- RGB-D и IMU backend D435i для Gazebo Harmonic. -->
+  <xacro:include
+    filename="$(find rtk2026_description)/urdf/sensors/realsense_d435i_gazebo.xacro"/>
   <!-- ROBOT PARAMETERS  -->
   <xacro:property name="base_mass" value="1.6"/>
@@ -53,5 +59,4 @@
   <xacro:property name="imu_height" value="0.01"/>
   <xacro:property name="lidar_height" value="0.040"/>
-  <xacro:property name="camera_depth" value="0.025"/>
   <!-- PHYSICAL ROBOT -->
   <xacro:rtk2026_diffbot_base
@@ -86,4 +91,13 @@
     use_mesh="false"
     mesh=""/>
+  <!--
+    Gazebo IMU публикует ориентацию, angular velocity и linear acceleration.
+    EKF использует только angular_velocity.z; абсолютный yaw не объединяем.
+  -->
+  <xacro:rtk2026_imu_gazebo
+    prefix="$(arg prefix)"
+    update_rate="100.0"
+    angular_velocity_stddev="0.002"
+    linear_acceleration_stddev="0.02"/>
   <!-- Лидар сверху в геометрическом центре корпуса. -->
   <xacro:rtk2026_lidar
@@ -106,14 +120,19 @@
     range_resolution="0.01"
     noise_stddev="0.005"/>
-  <!-- Камера по центру передней грани; пока только геометрия и TF-фреймы. -->
-  <xacro:rtk2026_webcam
-    prefix="$(arg prefix)"
+  <!--
+    D435i установлена по центру передней грани.
+    origin задаёт положение нижнего резьбового крепления официальной модели.
+    Смещение -12.5 мм по Z оставляет оптические центры на средней высоте
+    корпуса. Все внутренние смещения color/depth/infra/IMU берутся из
+    realsense2_description и здесь не дублируются.
+  -->
+  <xacro:sensor_d435i
     parent="$(arg prefix)base_link"
-    xyz="${base_length/2.0 + camera_depth/2.0} 0 0"
-    rpy="0 0 0"
-    mass="0.035"
-    width="0.060"
-    height="0.025"
-    depth="${camera_depth}"/>
+    name="$(arg prefix)camera"
+    use_nominal_extrinsics="true">
+    <origin xyz="${base_length/2.0} 0 -0.0125" rpy="0 0 0"/>
+  </xacro:sensor_d435i>
+  <xacro:rtk2026_realsense_d435i_gazebo
+    name="$(arg prefix)camera"/>
   <!-- ROS 2 CONTROL  -->
   <xacro:rtk2026_diffbot_ros2_control

File: src/rtk2026_description/urdf/sensors/webcam_gazebo.xacro (robot description, xacro)
@@ -10,10 +10,12 @@
       horizontal_fov — горизонтальный угол обзора в радианах.
     Для Gazebo Sim изображение публикуется сначала в Gazebo Transport и
-    требует отдельного ros_gz_bridge. Макрос не вызывается текущей
-    rtk2026_diff_drive_sim.urdf.xacro и оставлен как готовая точка расширения.
+    передаётся в ROS 2 через ros_gz_bridge из sim_slam_launch.py.
   -->
   <xacro:macro name="rtk2026_webcam_gazebo" params="prefix backend width height update_rate horizontal_fov">
+    <!-- Сохраняем отдельный физический camera_link после URDF -> SDF. -->
+    <gazebo reference="${prefix}camera_joint">
+      <preserveFixedJoint>true</preserveFixedJoint>
+    </gazebo>
     <gazebo reference="${prefix}camera_link">
-      <preserveFixedJoint>true</preserveFixedJoint>
       <sensor name="${prefix}webcam_sensor" type="camera">
         <always_on>true</always_on>
@@ -21,4 +23,5 @@
         <update_rate>${update_rate}</update_rate>
         <topic>${prefix}webcam/image_raw</topic>
+        <gz_frame_id>${prefix}camera_optical_frame</gz_frame_id>
         <camera>
           <horizontal_fov>${horizontal_fov}</horizontal_fov>
