Commit message: Вернуть body_x реальной модели, снизить крейсерскую скорость Nav2
body_x. При переносе точки отсчёта корпуса с base_footprint на ось
привода пересчитали только Z (0.080 - 0.060 = 0.020), а X молча
обнулили - хотя смена отсчёта чисто вертикальная и X не касается.
Силуэт в RViz был сдвинут вперёд на 60 мм относительно footprint в
nav2_params.yaml и реальной геометрии гусениц; на TF и Pi это не
влияло, только на картинку и на сверку с costmap.

footprint. Сверен с реальным URDF: track_end_x и track_radius
совпадают день в день, отсюда те же границы по X. По Y небольшое
расхождение - track_width реальной модели 0.025 против 0.033 у
tracked_sim, то есть footprint шире робота на 4 мм на сторону.
Направление безопасное, footprint_padding (5 мм) и так перекрывает
разницу - не трогал, только задокументировал.

Скорость. desired_linear_vel 0.24 -> 0.15 м/с - тот же порядок, что
рекомендован для ручного проезда при картографировании. Аппаратный
потолок (max_linear_mps 0.586 в arduino_bridge.yaml) далеко не задет,
ограничение чисто программное. Вместе с ним пропорционально снижены
зависимые пороги: min_approach_linear_velocity, regulated_linear_
scaling_min_speed, rotate_to_heading_angular_vel в FollowPath и
max_rotational_vel/min_rotational_vel/rotational_acc_lim в
behavior_server.

File: src/rtk2026_description/urdf/rtk2026_real.urdf.xacro (robot description, xacro)
@@ -121,7 +121,13 @@
     В гусеничной модели корпус отсчитывался от base_footprint и стоял на
     (-0.060, 0, 0.080) при оси на высоте 0.060. Здесь начало отсчёта -
-    сама ось, поэтому по Z остаётся 0.080 - 0.060 = 0.020.
-  -->
-  <xacro:property name="body_x" value="0"/>
+    сама ось, поэтому по Z остаётся 0.080 - 0.060 = 0.020. Смена точки
+    отсчёта чисто вертикальная и X не касается: он переносится как есть,
+    -0.060 - корпус на 60 мм ближе к заднему катку, чем к переднему.
+    Раньше здесь стоял 0 - X обнулили заодно с пересчётом Z, хотя ось
+    привода на X никак не влияет. Из-за этого силуэт в RViz был сдвинут
+    вперёд на 60 мм и не совпадал с footprint в nav2_params.yaml, который
+    взят из той же гусеничной модели и остался несимметричным.
+  -->
+  <xacro:property name="body_x" value="-0.060"/>
   <xacro:property name="body_z" value="0.020"/>
   <!-- Гусеница. Числа из гусеничной модели. -->
