Commit message: Set the robot envelope to 310 mm and place the footprint at the axle
base_footprint sits on the ground under the drive axle, not at the centre
of the robot — the body is offset 60 mm back and 80 mm up. The footprint I
committed earlier was centred on the frame, so Nav2 believed the robot
reached 60 mm further forward than it does and 60 mm less to the rear. On an
800 mm road that is the difference between clearing a turn and clipping it.
The rectangle is asymmetric now: x from -0.215 to +0.095.

The overall length also came from the wrong part. The body box is 300 mm,
but the track idler wheels stood 30 mm past it at each end, so the real
envelope was 360 mm. Target is 310 mm overall, so the wheels move in to
±0.095 from the track centre and the track box shrinks to 190 mm; the body
stays 300 mm and now sits just inside the envelope.

The track box length is derived from track_end_x in the xacro instead of
being written out again, since two numbers that must agree will not.

Verified the footprint equals the model's collision extents exactly, in
both costmaps, and that the xacro and the SDF give the same 310 x 246 mm.

File: src/rtk2026_tracked_sim/urdf/rtk2026_tracked.urdf.xacro (robot description, xacro)
@@ -15,8 +15,12 @@
   <xacro:property name="base_length" value="0.300"/>
   <!--
-    Полный поперечный габарит равен 240 мм:
+    Полный поперечный габарит равен 246 мм:
       корпус 180 мм;
-      две гусеницы по 30 мм;
-      средние плоскости гусениц разнесены на 210 мм.
+      две гусеницы по 33 мм;
+      средние плоскости гусениц разнесены на 213 мм.
+    Продольный габарит 310 мм задают не корпус, а колёса гусениц:
+      корпус 300 мм, от -0.210 до +0.090 от оси привода;
+      колёса от -0.215 до +0.095.
+    В footprint для Nav2 идёт наружный, то есть 310 мм.
   -->
   <xacro:property name="base_width" value="0.180"/>
@@ -27,5 +31,5 @@
   <xacro:property name="track_width" value="0.033"/>
   <xacro:property name="track_radius" value="0.060"/>
-  <xacro:property name="track_end_x" value="0.120"/>
+  <xacro:property name="track_end_x" value="0.095"/>
   <link name="base_footprint"/>
   <link name="base_link">
@@ -53,5 +57,5 @@
         <origin xyz="0 0 -0.020" rpy="0 0 0"/>
         <geometry>
-          <box size="0.240 ${track_width} 0.080"/>
+          <box size="${2.0 * track_end_x} ${track_width} 0.080"/>
         </geometry>
         <material name="${side}_track_black">
